File: Backplane Files/Cards/Power_Control_Card/Power_Control_Card.kicad_sch (KiCad schematic)
At the start: 17 parts, among them J1 Conn_01x02, Q1 FQPF27P06

Commit message: adding 3d models
Parts:
- J1: footprint Connector_PinHeader_2.54mm:PinHeader_1x02_P2.54mm_Vertical -> Connector_JST:JST_PH_B2B-PH-K_1x02_P2.00mm_Vertical
